Commit message: Changed arm model to the one used in ROS2 driver

File: spot_description/urdf/spot_arm.xacro (robot description, xacro)
@@ -1,220 +1,212 @@
-<?xml version="1.0" ?>
-<robot name="spot_arm" xmlns:xacro="http://www.ros.org/wiki/xacro">
-<material name="silver">
-  <color rgba="0.700 0.700 0.700 1.000"/>
-</material>
-<link name="base_arm_link">
-  <inertial>
-    <origin rpy="0 0 0" xyz="1.2371844231029972e-17 0.0 0.0325"/>
-    <mass value="5.770791545379091"/>
-    <inertia ixx="0.007226" ixy="-0.0" ixz="0.0" iyy="0.007226" iyz="0.0" izz="0.010387"/>
-  </inertial>
-  <visual>
-    <origin rpy="0 0 0" xyz="0 0 0"/>
-    <geometry>
-      <mesh filename="package://spot_description/meshes/arm/base_link.stl" scale="0.001 0.001 0.001"/>
-    </geometry>
-    <material name="silver"/>
-  </visual>
-  <collision>
-    <origin rpy="0 0 0" xyz="0 0 0"/>
-    <geometry>
-      <mesh filename="package://spot_description/meshes/arm/base_link.stl" scale="0.001 0.001 0.001"/>
-    </geometry>
-  </collision>
-</link>
-<link name="link4">
-  <inertial>
-    <origin rpy="0 0 0" xyz="-0.00911464892336129 0.12606054498393937 5.551115123125783e-17"/>
-    <mass value="10.95245995004642"/>
-    <inertia ixx="0.066789" ixy="0.011971" ixz="-0.0" iyy="0.014993" iyz="0.0" izz="0.071949"/>
-  </inertial>
-  <visual>
-    <origin rpy="0 0 0" xyz="0.001 -0.4505 -0.0475"/>
-    <geometry>
-      <mesh filename="package://spot_description/meshes/arm/link4.stl" scale="0.001 0.001 0.001"/>
-    </geometry>
-    <material name="silver"/>
-  </visual>
-  <collision>
-    <origin rpy="0 0 0" xyz="0.001 -0.4505 -0.0475"/>
-    <geometry>
-      <mesh filename="package://spot_description/meshes/arm/link4.stl" scale="0.001 0.001 0.001"/>
-    </geometry>
-  </collision>
-</link>
-<link name="gripper">
-  <inertial>
-    <origin rpy="0 0 0" xyz="-8.366123908053191e-08 0.07051371901138614 0.017123167388316526"/>
-    <mass value="5.9780007036604434"/>
-    <inertia ixx="0.01723" ixy="0.0" ixz="0.0" iyy="0.00734" iyz="-0.003871" izz="0.0153"/>
-  </inertial>
-  <visual>
-    <origin rpy="0 0 0" xyz="0.0085 -0.77959 -0.0475"/>
-    <geometry>
-      <mesh filename="package://spot_description/meshes/arm/gripper.stl" scale="0.001 0.001 0.001"/>
-    </geometry>
-    <material name="silver"/>
-  </visual>
-  <collision>
-    <origin rpy="0 0 0" xyz="0.0085 -0.77959 -0.0475"/>
-    <geometry>
-      <mesh filename="package://spot_description/meshes/arm/gripper.stl" scale="0.001 0.001 0.001"/>
-    </geometry>
-  </collision>
-</link>
-<link name="finger">
-  <inertial>
-    <origin rpy="0 0 0" xyz="0.8635899028063472 0.09862056591557622 0.00850232975194119"/>
-    <mass value="1.71236178687828"/>
-    <inertia ixx="0.002129" ixy="0.0" ixz="-0.0" iyy="0.001681" iyz="0.000162" izz="0.003403"/>
-  </inertial>
-  <visual>
-    <origin rpy="0 0 0" xyz="0.87709 -0.823505 -0.0185"/>
-    <geometry>
-      <mesh filename="package://spot_description/meshes/arm/finger.stl" scale="0.001 0.001 0.001"/>
-    </geometry>
-    <material name="silver"/>
-  </visual>
-  <collision>
-    <origin rpy="0 0 0" xyz="0.87709 -0.823505 -0.0185"/>
-    <geometry>
-      <mesh filename="package://spot_description/meshes/arm/finger.stl" scale="0.001 0.001 0.001"/>
-    </geometry>
-  </collision>
-</link>
-<link name="link2">
-  <inertial>
-    <origin rpy="0 0 0" xyz="-0.0163095589512068 0.17540914221218962 0.0"/>
-    <mass value="12.658281999999998"/>
-    <inertia ixx="0.12979" ixy="0.002625" ixz="0.0" iyy="0.01004" iyz="0.0" izz="0.129493"/>
-  </inertial>
-  <visual>
-    <origin rpy="0 0 0" xyz="-0.015 -0.0 -0.115"/>
-    <geometry>
-      <mesh filename="package://spot_description/meshes/arm/link2.stl" scale="0.001 0.001 0.001"/>
-    </geometry>
-    <material name="silver"/>
-  </visual>
-  <collision>
-    <origin rpy="0 0 0" xyz="-0.015 -0.0 -0.115"/>
-    <geometry>
-      <mesh filename="package://spot_description/meshes/arm/link2.stl" scale="0.001 0.001 0.001"/>
-    </geometry>
-  </collision>
-</link>
-<link name="link1">
-  <inertial>
-    <origin rpy="0 0 0" xyz="0.05071972800114364 -1.0308563411658574e-17 0.04676911608650795"/>
-    <mass value="6.925827706354272"/>
-    <inertia ixx="0.01241" ixy="-0.0" ixz="-0.001047" iyy="0.010387" iyz="0.0" izz="0.012306"/>
-  </inertial>
-  <visual>
-    <origin rpy="0 0 0" xyz="-0.0 -0.0 -0.065"/>
-    <geometry>
-      <mesh filename="package://spot_description/meshes/arm/link1.stl" scale="0.001 0.001 0.001"/>
-    </geometry>
-    <material name="silver"/>
-  </visual>
-  <collision>
-    <origin rpy="0 0 0" xyz="-0.0 -0.0 -0.065"/>
-    <geometry>
-      <mesh filename="package://spot_description/meshes/arm/link1.stl" scale="0.001 0.001 0.001"/>
-    </geometry>
-  </collision>
-</link>
-<link name="wrist">
-  <inertial>
-    <origin rpy="0 0 0" xyz="0.03954999709763633 0.03472006124891969 4.209155544249166e-08"/>
-    <mass value="3.2278801394086396"/>
-    <inertia ixx="0.00339" ixy="-2.1e-05" ixz="0.0" iyy="0.002242" iyz="-0.0" izz="0.003439"/>
-  </inertial>
-  <visual>
-    <origin rpy="0 0 0" xyz="0.0485 -0.69859 -0.0475"/>
-    <geometry>
-      <mesh filename="package://spot_description/meshes/arm/wrist.stl" scale="0.001 0.001 0.001"/>
-    </geometry>
-    <material name="silver"/>
-  </visual>
-  <collision>
-    <origin rpy="0 0 0" xyz="0.0485 -0.69859 -0.0475"/>
-    <geometry>
-      <mesh filename="package://spot_description/meshes/arm/wrist.stl" scale="0.001 0.001 0.001"/>
-    </geometry>
-  </collision>
-</link>
-<link name="link3">
-  <inertial>
-    <origin rpy="0 0 0" xyz="-0.015621881612358529 0.06665620790957599 -0.058074231003688394"/>
-    <mass value="7.368455487741179"/>
-    <inertia ixx="0.018073" ixy="0.000915" ixz="-0.00101" iyy="0.011789" iyz="0.003728" izz="0.01667"/>
-  </inertial>
-  <visual>
-    <origin rpy="0 0 0" xyz="-0.017 -0.3125 -0.115"/>
-    <geometry>
-      <mesh filename="package://spot_description/meshes/arm/link3.stl" scale="0.001 0.001 0.001"/>
-    </geometry>
-    <material name="silver"/>
-  </visual>
-  <collision>
-    <origin rpy="0 0 0" xyz="-0.017 -0.3125 -0.115"/>
-    <geometry>
-      <mesh filename="package://spot_description/meshes/arm/link3.stl" scale="0.001 0.001 0.001"/>
-    </geometry>
-  </collision>
-</link>
-<joint name="base_arm_joint" type="fixed">
-        <origin xyz="0.29 0 0.08" rpy="0 0 0" />
-        <parent link="body" />
-        <child link="base_arm_link" />
-    </joint>
-<joint name="arm_joint1" type="revolute">
-  <origin rpy="0 0 0" xyz="0.0 0.0 0.065"/>
-  <parent link="base_arm_link"/>
-  <child link="link1"/>
-  <axis xyz="0.0 0.0 1.0"/>
-  <limit effort="100" lower="-3.141593" upper="2.617994" velocity="100"/>
-</joint>
-<joint name="arm_joint2" type="revolute">
-  <origin rpy="0 0 0" xyz="0.015 0.0 0.05"/>
-  <parent link="link1"/>
-  <child link="link2"/>
-  <axis xyz="-1.0 0.0 0.0"/>
-  <limit effort="100" lower="-3.665191" upper="0.0" velocity="100"/>
-</joint>
-<joint name="arm_joint3" type="revolute">
-  <origin rpy="0 0 0" xyz="0.002 0.3125 0.0"/>
-  <parent link="link2"/>
-  <child link="link3"/>
-  <axis xyz="1.0 0.0 0.0"/>
-  <limit effort="100" lower="0.0" upper="2.96706" velocity="100"/>
-</joint>
-<joint name="arm_joint4" type="revolute">
-  <origin rpy="0 0 0" xyz="-0.018 0.138 -0.0675"/>
-  <parent link="link3"/>
-  <child link="link4"/>
-  <axis xyz="0.0 1.0 0.0"/>
-  <limit effort="100" lower="-2.879793" upper="2.879793" velocity="100"/>
-</joint>
-<joint name="arm_joint5" type="revolute">
-  <origin rpy="0 0 0" xyz="-0.0475 0.24809 0.0"/>
-  <parent link="link4"/>
-  <child link="wrist"/>
-  <axis xyz="1.0 0.0 0.0"/>
-  <limit effort="100" lower="-1.570796" upper="1.570796" velocity="100"/>
-</joint>
-<joint name="arm_joint6" type="revolute">
-  <origin rpy="0 0 0" xyz="0.04 0.081 0.0"/>
-  <parent link="wrist"/>
-  <child link="gripper"/>
-  <axis xyz="-0.0 1.0 0.0"/>
-  <limit effort="100" lower="-2.96706" upper="2.96706" velocity="100"/>
-</joint>
-<joint name="arm_gripper" type="revolute">
-  <origin rpy="0 0 0" xyz="-0.86859 0.043915 -0.029"/>
-  <parent link="gripper"/>
-  <child link="finger"/>
-  <axis xyz="1.0 -0.0 0.0"/>
-  <limit effort="100" lower="-1.396263" upper="0.349066" velocity="100"/>
-</joint>
+<?xml version="1.0"?>
+<robot name="spot_arm">
+  <link name="arm_link_sh0">
+    <visual>
+      <origin xyz="0 0 0" rpy="0 0 0"/>
+      <geometry>
+        <mesh filename="package://spot_description/meshes/arm/visual/arm_link_sh0.obj"/>
+      </geometry>
+      <material name="arm_link_sh0"> <color rgba="0.2 0.2 0.2 1"/></material>
+    </visual>
+    <collision>
+      <geometry>
+        <mesh filename="package://spot_description/meshes/arm/collision/arm_link_sh0.stl" />
+      </geometry>
+    </collision>
+    <inertial>
+      <origin rpy="0.0013490340912847287 -0.15433618253071657 0.0066354181456347305" xyz="-0.012372709810733795 -4.5211403630673885e-05 -0.02103196457028389"/>
+      <mass value="2.3364000000000003"/>
+      <inertia ixx="0.009014303010689815" ixy="0.0" ixz="0.0" iyy="0.005835102417829581" iyz="0.0" izz="0.00778747846359954"/>
+    </inertial>
+  </link>
+  <joint name="arm_joint1" type="revolute">
+    <origin xyz="0.292 0.0 0.188" rpy="0 0 0"/>
+    <axis xyz="0 0 1"/>
+    <parent link="body"/>
+    <child link="arm_link_sh0"/>
+    <limit effort="1000" velocity="1000.00" lower="-2.61799387799149441136" upper="3.14159265358979311599"/>
+  </joint>
+  <link name="arm_link_sh1">
+    <visual>
+      <origin xyz="0 0 0" rpy="0 0 0"/>
+      <geometry>
+        <mesh filename="package://spot_description/meshes/arm/visual/arm_link_sh1.obj"/>
+      </geometry>
+      <material name="arm_link_sh1"> <color rgba="0.2 0.2 0.2 1"/></material>
+    </visual>
+    <collision>
+      <geometry>
+        <mesh filename="package://spot_description/meshes/arm/collision/arm_link_sh1.stl" />
+      </geometry>
+    </collision>
+    <inertial>
+      <origin rpy="0.009910032200701302 -0.5123007314267984 0.002209016500439809" xyz="2.4176391889341176e-05 2.4116111490002368e-06 -1.0059113265015185e-05"/>
+      <mass value="0.2596"/>
+      <inertia ixx="0.00020292766231464653" ixy="0.0" ixz="0.0" iyy="0.00017078637725384855" iyz="0.0" izz="0.00020384964230406682"/>
+    </inertial>
+  </link>
+  <joint name="arm_joint2" type="revolute">
+    <origin xyz="0.0 0.0 0.0" rpy="0 0 0"/>
+    <axis xyz="0 1 0"/>
+    <parent link="arm_link_sh0"/>
+    <child link="arm_link_sh1"/>
+    <!-- <limit effort="1000" velocity="1000.00" lower="-0.52359877559829881565" upper="3.14159265358979311599"/> -->
+    <limit effort="1000" velocity="1000.00" lower="-3.14159265358979311599" upper="0.52359877559829881565"/>
+  </joint>
+  <link name="arm_link_hr0">
+    <visual>
+      <origin xyz="0 0 0" rpy="0 0 0"/>
+      <geometry>
+        <mesh filename="package://spot_description/meshes/arm/visual/arm_link_hr0.obj"/>
+      </geometry>
+      <material name="arm_link_hr0"> <color rgba="0.2 0.2 0.2 1"/></material>
+    </visual>
+    <collision>
+      <geometry>
+        <mesh filename="package://spot_description/meshes/arm/collision/arm_link_hr0.stl" />
+      </geometry>
+    </collision>
+    <inertial>
+      <origin rpy="-0.01179850657706405 0.0002834144901480151 -0.02372295500868482" xyz="0.17047011852264404 -0.0019251034827902913 4.483893280848861e-05"/>
+      <mass value="1e-06"/>
+      <inertia ixx="6.312631747339145e-10" ixy="0.0" ixz="0.0" iyy="1.1487063558949979e-08" iyz="0.0" izz="1.161105128440526e-08"/>
+    </inertial>
+  </link>
+  <joint name="arm_hr0" type="fixed">
+    <origin xyz="0.0 0.0 0.0" rpy="0 0 0"/>
+    <axis xyz="1 0 0"/>
+    <parent link="arm_link_sh1"/>
+    <child link="arm_link_hr0"/>
+    <limit effort="1000" velocity="1000.00" lower="-1e6" upper="1e6"/>
+  </joint>
+  <link name="arm_link_el0">
+    <visual>
+      <origin xyz="0 0 0" rpy="0 0 0"/>
+      <geometry>
+        <mesh filename="package://spot_description/meshes/arm/visual/arm_link_el0.obj"/>
+      </geometry>
+      <material name="arm_link_el0"> <color rgba="0.2 0.2 0.2 1"/></material>
+    </visual>
+    <collision>
+      <geometry>
+        <mesh filename="package://spot_description/meshes/arm/collision/arm_link_el0.stl" />
+      </geometry>
+    </collision>
+    <inertial>
+      <origin rpy="-0.004185887288594259 -0.6136269547775202 -0.0004619387581783485" xyz="0.0553741455078125 0.00023603376757819206 0.04827198013663292"/>
+      <mass value="0.725"/>
+      <inertia ixx="0.0008215365829160558" ixy="0.0" ixz="0.0" iyy="0.0020047889807066404" iyz="0.0" izz="0.0019722797759789395"/>
+    </inertial>
+  </link>
+  <joint name="arm_joint3" type="revolute">
+    <origin xyz="0.3385 0 0" rpy="0 0 0"/>
+    <axis xyz="0 1 0"/>
+    <parent link="arm_link_hr0"/>
+    <child link="arm_link_el0"/>
+    <limit effort="1000" velocity="1000.00" lower="0" upper="3.14159265358979311599"/>
+  </joint>
+  <link name="arm_link_el1">
+    <visual>
+      <origin xyz="0 0 0" rpy="0 0 0"/>
+      <geometry>
+        <mesh filename="package://spot_description/meshes/arm/visual/arm_link_el1.obj"/>
+      </geometry>
+      <material name="arm_link_el1"> <color rgba="0.2 0.2 0.2 1"/></material>
+    </visual>
+    <collision>
+      <geometry>
+        <mesh filename="package://spot_description/meshes/arm/collision/arm_link_el1.stl" />
+      </geometry>
+    </collision>
+    <inertial>
+      <origin rpy="-0.15027374227250867 -0.0007874585461915551 0.003728225436950172" xyz="-0.1257835328578949 -0.013684478588402271 0.00010157923679798841"/>
+      <mass value="0.725"/>
+      <inertia ixx="0.0006254807525240598" ixy="0.0" ixz="0.0" iyy="0.004402454711936095" iyz="0.0" izz="0.004515915146038191"/>
+    </inertial>
+  </link>
+  <joint name="arm_joint4" type="revolute">
+    <origin xyz="0.40330 0.0 0.0750" rpy="0 0 0"/>
+    <axis xyz="1 0 0"/>
+    <parent link="arm_link_el0"/>
+    <child link="arm_link_el1"/>
+    <limit effort="1000" velocity="1000.00" lower="-2.79252680319092716487" upper="2.79252680319092716487"/>
+  </joint>
+  <link name="arm_link_wr0">
+    <visual>
+      <origin xyz="0 0 0" rpy="0 0 0"/>
+      <geometry>
+        <mesh filename="package://spot_description/meshes/arm/visual/arm_link_wr0.obj"/>
+      </geometry>
+      <material name="arm_link_wr0"> <color rgba="0.2 0.2 0.2 1"/></material>
+    </visual>
+    <collision>
+      <geometry>
+        <mesh filename="package://spot_description/meshes/arm/collision/arm_link_wr0.stl" />
+      </geometry>
+    </collision>
+    <inertial>
+      <origin rpy="-0.4951534907966386 0.0033720434077784134 0.020027599337697932" xyz="0.008210677653551102 -0.012051000259816647 3.143483627354726e-05"/>
+      <mass value="0.98"/>
+      <inertia ixx="0.0009851320696685427" ixy="0.0" ixz="0.0" iyy="0.0008916145765810678" iyz="0.0" izz="0.0012354892751854467"/>
+    </inertial>
+  </link>
+  <joint name="arm_joint5" type="revolute">
+    <origin xyz="0.0 0.0 0.0" rpy="0 0 0"/>
+    <axis xyz="0 1 0"/>
+    <parent link="arm_link_el1"/>
+    <child link="arm_link_wr0"/>
+    <limit effort="1000" velocity="1000.00" lower="-1.83259571459404613236" upper="1.83259571459404613236"/>
+  </joint>
+  <link name="arm_link_wr1">
+    <visual>
+      <origin xyz="0 0 0" rpy="0 0 0"/>
+      <geometry>
+        <mesh filename="package://spot_description/meshes/arm/visual/arm_link_wr1.obj"/>
+      </geometry>
+      <material name="arm_link_wr1"> <color rgba="0.2 0.2 0.2 1"/></material>
+    </visual>
+    <collision>
+      <geometry>
+        <mesh filename="package://spot_description/meshes/arm/collision/arm_link_wr1.stl" />
+      </geometry>
+    </collision>
+    <inertial>
+      <origin rpy="0.006393076449033863 0.2928526604761865 -0.022814984050994802" xyz="0.12516802549362183 0.00010137435310753062 -0.013997982256114483"/>
+      <mass value="0.785"/>
+      <inertia ixx="0.00076741362048185" ixy="0.0" ixz="0.0" iyy="0.0017628124054271809" iyz="0.0" izz="0.0016818105865345951"/>
+    </inertial>
+  </link>
+  <joint name="arm_joint6" type="revolute">
+    <origin xyz="0.0 0.0 0.0" rpy="0 0 0"/>
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